File: lets_split/lets_split.kicad_pcb (KiCad board)
At the start: 2 copper layers, 112 x 79 mm, 62 parts, among them J1 3PIN, J2 6PIN, J3 3PIN, SW1 SW_PUSH, SW10 SW_PUSH, SW11 SW_PUSH, SW12 SW_PUSH, SW13 SW_PUSH, SW14 SW_PUSH, SW15 SW_PUSH, SW16 SW_PUSH, SW17 SW_PUSH, SW18 SW_PUSH, SW19 SW_PUSH, SW2 SW_PUSH, SW21 SW_PUSH, SW22 SW_PUSH, SW23 SW_PUSH, SW3 SW_PUSH, SW4 SW_PUSH, SW5 SW_PUSH, SW6 SW_PUSH, SW7 SW_PUSH, SW8 SW_PUSH, SW9 SW_PUSH, U2 HOLE, U3 HOLE, U4 HOLE, U5 HOLE

Commit message: New version of the project added.
Parts:
- removed the G*** at (118.8, 78.0)
- removed the G*** at (127.0, 87.8)
- removed J2: 6PIN, footprint:4pin35mmAudio
- added ?: , SparkFun-Connectors:AUDIO-JACK-TRRS-SMD, B.Cu at (131.3, 36.0)
- added ?: SolderWirePad_single_SMD_5x10mm, Wire_Pads:SolderWirePad_single_SMD_5x10mm, B.Cu at (127.4, 76.4)
- added ?: SolderWirePad_single_SMD_5x10mm, Wire_Pads:SolderWirePad_single_SMD_5x10mm, F.Cu at (51.4, 49.8)
- added ?: SolderWirePad_single_SMD_5x10mm, Wire_Pads:SolderWirePad_single_SMD_5x10mm, F.Cu at (51.4, 52.6)
- added ?: SolderWirePad_single_SMD_5x10mm, Wire_Pads:SolderWirePad_single_SMD_5x10mm, F.Cu at (71.2, 69.6)
- added ?: SolderWirePad_single_SMD_5x10mm, Wire_Pads:SolderWirePad_single_SMD_5x10mm, B.Cu at (71.2, 69.6)
- added ?: , SparkFun-Connectors:AUDIO-JACK-TRRS-SMD, F.Cu at (131.3, 36.0)
- added ?: SolderWirePad_single_SMD_5x10mm, Wire_Pads:SolderWirePad_single_SMD_5x10mm, B.Cu at (51.4, 49.8)
- added ?: SolderWirePad_single_SMD_5x10mm, Wire_Pads:SolderWirePad_single_SMD_5x10mm, B.Cu at (51.4, 52.6)
- added ?: SolderWirePad_single_SMD_5x10mm, Wire_Pads:SolderWirePad_single_SMD_5x10mm, F.Cu at (127.4, 77.0)
- added ?: SolderWirePad_single_SMD_5x10mm, Wire_Pads:SolderWirePad_single_SMD_5x10mm, B.Cu at (127.4, 73.3)
- added ?: SolderWirePad_single_SMD_5x10mm, Wire_Pads:SolderWirePad_single_SMD_5x10mm, F.Cu at (127.4, 74.0)
- added ?: SolderWirePad_single_SMD_5x10mm, Wire_Pads:SolderWirePad_single_SMD_5x10mm, B.Cu at (127.4, 70.5)
- added ?: SolderWirePad_single_SMD_5x10mm, Wire_Pads:SolderWirePad_single_SMD_5x10mm, F.Cu at (127.4, 71.1)
- added G***: LOGO, picLIB:heart_4mm, F.Cu at (145.9, 109.2)
- added G***: LOGO, picLIB:RandM_29x39mm, F.Cu at (51.8, 72.4)
- added G***: LOGO, picLIB:robot_34mm, B.Cu at (78.0, 94.4)
- added G***: LOGO, picLIB:picklerick_9x21mm, B.Cu at (109.7, 96.0)
- added G***: LOGO, picLIB:illuminati_10mm, F.Cu at (142.2, 93.2)
- added G***: LOGO, picLIB:heart_4mm, B.Cu at (115.6, 108.9)
- added REF**: MountingHole_2.2mm_M2, Mounting_Holes:MountingHole_2.2mm_M2, F.Cu at (131.3, 44.6)
- added REF**: MountingHole_2.2mm_M2, Mounting_Holes:MountingHole_2.2mm_M2, F.Cu at (131.3, 37.6)
- moved W1 31.5 mm to (96.3, 40.0), turned to 180 degrees
Routing:
- net Net-(U1-Pad29): track 0.00 -> 104.5 mm, vias 0 -> 7
- net xtradata: track 25.8 -> 90.8 mm, vias 0 -> 4
- net data: track 117.5 -> 83.3 mm, vias 0 -> 4
- net Net-(R1-Pad2): track 77.0 -> 61.2 mm
- net Net-(U1-Pad22): track 0.00 -> 11.6 mm
- net Net-(U1-Pad23): track 0.00 -> 11.4 mm
- net VCC: track 27.2 -> 37.7 mm, vias 0 -> 1
- net GND: track 15.8 -> 23.1 mm, vias 0 -> 1
- net Net-(J1-Pad2): track 19.5 -> 12.4 mm, vias 0 -> 1
- net (no net): track 6.60 -> 13.4 mm, vias 0 -> 2
- net row0: track 96.8 -> 100.5 mm
- net Net-(J2-Pad4): track 18.7 -> 21.7 mm, vias 0 -> 4
- net col1: track 68.7 -> 66.1 mm, vias 0 -> 1
- net Net-(D13-Pad2): track 6.57 -> 8.90 mm
- net Net-(D9-Pad2): track 6.67 -> 9.00 mm
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Other:
- board text added: "Din"
- board text added: "Made with"
- board text added: "data"
- board text removed: "By Wootpatoot"
- board text removed: "I2C"
