File: lets_split/lets_split.sch (KiCad schematic (older format))
At the start: 60 parts, among them J1 3PIN, J2 6PIN, J3 3PIN, SW1 SW_PUSH, SW10 SW_PUSH, SW11 SW_PUSH, SW12 SW_PUSH, SW13 SW_PUSH, SW14 SW_PUSH, SW15 SW_PUSH, SW16 SW_PUSH, SW17 SW_PUSH, SW18 SW_PUSH, SW19 SW_PUSH, SW2 SW_PUSH, SW20 SW_PUSH, SW21 SW_PUSH, SW22 SW_PUSH, SW23 SW_PUSH, SW24 SW_PUSH, SW3 SW_PUSH, SW4 SW_PUSH, SW5 SW_PUSH, SW6 SW_PUSH, SW7 SW_PUSH, SW8 SW_PUSH, SW9 SW_PUSH, U1 TEENSY2.0, U2 HOLE, U3 HOLE, U4 HOLE, U5 HOLE

Commit message: New version of the project added.
Parts:
- W1: symbol TEST -> TEST-RESCUE-lets_split
Changed lines of the file:
@@
 EESchema Schematic File Version 2
+LIBS:lets_split-rescue
 LIBS:power
 LIBS:device
@@
 LIBS:siliconi
 LIBS:opto
+LIBS:SparkFun-Connectors
 LIBS:atmel
 LIBS:contrib
 LIBS:valves
-LIBS:component
 LIBS:lets_split-cache
 EELAYER 25 0
@@
 xtradata
 $Comp
-L TEST W1
+L TEST-RESCUE-lets_split W1
 U 1 1 57D52188
 P 4400 900
